File: wirebonding-badge/wirebonding-badge.kicad_pcb (KiCad board)
At the start: 2 copper layers, 56.4 x 32.8 mm, 14 parts, among them SW1 SW_Push, SW2 SW_Push, SW3 SW_Push, SW4 SW_Push, U3 LM2576HVS-3.3

Commit message: Finished connections. Ready for prototyping.
Parts:
- removed U3: LM2576HVS-3.3, Package_TO_SOT_SMD:TO-263-5_TabPin3
- added U2: LM2576HVS-3.3, Package_TO_SOT_SMD:TO-263-5_TabPin3, F.Cu at (121.2, 101.9)
- SW1, SW2, SW3, SW4: footprint Button_Switch_THT:SW_PUSH_6mm -> Button_Switch_SMD:SW_Push_1TS009xxxx-xxxx-xxxx_6x6x5mm
- moved R1 5.28 mm to (146.8, 98.8), turned to 90 degrees
- moved C1 5.03 mm to (149.4, 98.8), turned to -90 degrees
- moved SW1 4.44 mm to (119.0, 84.6), turned to -90 degrees
- moved SW2 3.40 mm to (127.5, 84.5), turned to 90 degrees
- moved SW3 3.40 mm to (136.1, 84.5), turned to 90 degrees
- moved SW4 3.40 mm to (144.7, 84.5), turned to 90 degrees
Routing:
- net +3V0: track 4.59 -> 26.8 mm, vias 1 -> 7
- net Net-(U1-RST): track 8.25 -> 29.6 mm
- net Net-(U1-BUO2): track 7.71 -> 28.9 mm, vias 1 -> 2
- net Net-(U1-IO_A): track 8.42 -> 20.1 mm
- net Net-(U1-BUO1): track 7.13 -> 17.2 mm, vias 1 -> 2
- net Net-(U1-IO_C): track 8.72 -> 15.1 mm
- net Net-(U1-IO_B): track 8.74 -> 14.5 mm
- net Net-(U1-OSC): track 1.41 -> 3.78 mm
- added copper zone on B.Cu, net +3V0
Other:
- board text added: "."
- board text added: "U1"

Commit message: Final revision for 5/2025.
Parts:
- removed TP3, TP4: TestPoint, TestPoint:TestPoint_Keystone_5019_Minature
- added 10k-trim1: VR1, Resistor_SMD:TRIM_TC33X-2-102E, F.Cu at (133.2, 105.0)
- added C2: 100uF, Capacitor_SMD:C_1206_3216Metric, F.Cu at (128.4, 95.8)
- added C3: 330uF, Capacitor_SMD:C_1206_3216Metric, F.Cu at (117.0, 96.4)
- added C4: 1uF, Capacitor_SMD:C_1206_3216Metric, F.Cu at (139.4, 108.9)
- added C5: 1uF, Capacitor_SMD:C_1206_3216Metric, F.Cu at (139.5, 111.3)
- added C6: 10uF, Capacitor_SMD:C_1206_3216Metric, F.Cu at (160.9, 110.7)
- added C7: 220pF, Capacitor_SMD:C_1206_3216Metric, F.Cu at (155.6, 99.0)
- added C8: 220pF, Capacitor_SMD:C_1206_3216Metric, F.Cu at (160.2, 99.2)
- added D1: SD1206S040S1R0, Diode_SMD:D_1206_3216Metric_Pad1.42x1.75mm_HandSolder, F.Cu at (122.8, 96.6)
- added FB1: Ferrite, Inductor_SMD:L_1206_3216Metric_Pad1.22x1.90mm_HandSolder, F.Cu at (153.0, 99.2)
- added FB2: Ferrite, Inductor_SMD:L_1206_3216Metric_Pad1.22x1.90mm_HandSolder, F.Cu at (162.8, 99.4)
- added G***: LOGO, Library:logo_chippie, F.Cu at (141.5, 66.0)
- added G***: LOGO, Library:logo_hybond, F.Cu at (160.0, 61.0)
- added G***: LOGO, Library:logo_siliconinsider, F.Cu at (123.5, 61.0)
- added G***: LOGO, Library:logo_microq_greyscale, F.Cu at (124.0, 73.5)
- added G***: LOGO, Library:logo_texplained, F.Cu at (159.5, 72.0)
- added G***: LOGO, Library:logo_hardwareio, F.Cu at (141.5, 53.0)
- added L1: 330uH, Inductor_SMD:L_1206_3216Metric_Pad1.22x1.90mm_HandSolder, F.Cu at (121.4, 92.6)
- added R2: 100, Resistor_SMD:R_1206_3216Metric, F.Cu at (144.6, 108.9)
- added R3: 100, Resistor_SMD:R_1206_3216Metric, F.Cu at (144.6, 111.3)
- added R4: 10k, Resistor_SMD:R_1206_3216Metric, F.Cu at (157.9, 114.3)
- added U3: PAM8302AAS, Package_SO:MSOP-8_3x3mm_P0.65mm, F.Cu at (151.1, 110.3)
- LS1: footprint Buzzer_Beeper:Speaker_CUI_CMR-1206S-67 -> Buzzer_Beeper:same_sky_speaker_mix
- SW1: value SW_Push -> PCM12SMTR; footprint Button_Switch_SMD:SW_Push_1TS009xxxx-xxxx-xxxx_6x6x5mm -> Library:SW_PCM12SMTR
- moved TP1 13.2 mm to (166.2, 114.8)
- moved U2 8.00 mm to (121.4, 109.9)
- moved LS1 3.23 mm to (156.8, 88.0)
Connections:
- BT1 pad 1: +9V -> Net-(BT1-+)
- LS1 pad 1: Net-(U1-BUO1) -> Net-(C7-Pad2)
- LS1 pad 2: Net-(U1-BUO2) -> Net-(C8-Pad2)
- SW1 pad 1: GND -> Net-(BT1-+)
- SW1 pad 2: Net-(U1-RST) -> +9V
- U1 pad 7: Net-(U1-RST) -> +3V0
- U2 pad 2: unconnected-(U2-OUT-Pad2) -> Net-(D1-K)
- U2 pad 5: unconnected-(U2-~{ON}/OFF-Pad5) -> GND
Routing:
- net +3V0: track 26.8 -> 81.0 mm, vias 7 -> 12
- net Net-(BT1-+): track 0.00 -> 48.6 mm, vias 0 -> 1
- net Net-(U1-RST): track 29.6 -> 0.00 mm, vias 2 -> 0
- net Net-(C7-Pad2): track 0.00 -> 18.1 mm, vias 0 -> 2
- net Net-(C8-Pad2): track 0.00 -> 17.1 mm, vias 0 -> 2
- net Net-(U3-OUT-): track 0.00 -> 16.3 mm
- net GND: track 3.42 -> 17.6 mm, vias 1 -> 0
- net Net-(U3-OUT+): track 0.00 -> 11.7 mm
- net Net-(D1-K): track 0.00 -> 10.6 mm
- net Net-(U3-~{SD}): track 0.00 -> 10.3 mm
- net +9V: track 0.00 -> 9.20 mm, vias 0 -> 2
- net Net-(10k-trim1-Pad2): track 0.00 -> 7.84 mm
- net Net-(U1-BUO2): track 28.9 -> 23.2 mm
- net Net-(U3-IN+): track 0.00 -> 3.68 mm
- net Net-(U3-IN-): track 0.00 -> 2.97 mm
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Other:
- board size 56.4 x 32.8 mm -> 56.4 x 67.8 mm
